Commit message: Additions to RL model. Push to agnostic model

File: src/robo_ag_rl/urdf/ElephantMyCobotPro600/mycobot_pro_600.urdf (robot description, URDF)
Before this commit: robot myCobotPro600, 7 links, 6 joints
Links:
- removed link base
- added link base_link; collision mesh filename=package://RoboAgRL/urdf/ElephantMyCobotPro600/base.stl; visual mesh filename=package://RoboAgRL/urdf/ElephantMyCobotPro600/base.stl
Joints:
- joint joint2_to_joint1: parent base -> base_link
